File: kicad/Balance_GVS/Balance_GVS.kicad_pcb (KiCad board)
At the start: 2 copper layers, 30 x 100 mm, 96 parts, among them J1 Conn_01x02_Pin, J10 I2C Header 2, J5 Conn_01x02_Pin, J6 Conn_01x03_Pin, J7 Conn_01x03_Pin, J8 Conn_01x05_Pin, J9 I2C Header 1, K1 AQY210S, Q3 2N3904, Q4 2N3904, SW2 EVQ-P7A01P, SW3 SW_Push, SW4 SW_Push, SW5 SW_Push, SW6 SW_Push, U1 ESP32-WROOM-32E, U10 INA219BxD, U11 LT1013DIP, U12 LT1013DIP, U3 OPA4313IPWR, U4 INA303A1IPW, U9 MCP4725xxx-xCH

Commit message: Fixed schematic warnings
Parts:
- added D1: LED, LED_SMD:LED_0603_1608Metric_Pad1.05x0.95mm_HandSolder, F.Cu at (174.2, 88.8)
- added D2: LED, LED_SMD:LED_0603_1608Metric_Pad1.05x0.95mm_HandSolder, F.Cu at (174.2, 91.4)
- added D3: LED, LED_SMD:LED_0603_1608Metric_Pad1.05x0.95mm_HandSolder, F.Cu at (180.8, 101.2)
- added D5: LED, LED_SMD:LED_0603_1608Metric_Pad1.05x0.95mm_HandSolder, F.Cu at (174.2, 94.0)
- added D6: LED, LED_SMD:LED_0603_1608Metric_Pad1.05x0.95mm_HandSolder, F.Cu at (174.2, 96.6)
- added J11: Conn_01x02_Pin, Connector_PinSocket_2.54mm:PinSocket_1x02_P2.54mm_Vertical, F.Cu at (174.3, 102.2)
- added J12: Conn_01x02_Pin, Connector_PinSocket_2.54mm:PinSocket_1x02_P2.54mm_Vertical, F.Cu at (178.7, 89.8)
- added J13: UART Header, Connector_PinSocket_2.54mm:PinSocket_1x02_P2.54mm_Vertical, F.Cu at (183.3, 89.8)
Connections:
- net 24V renamed +24V
- R45 pad 1: Net-(D5-A) -> Net-(D1-A)
- R46 pad 1: Net-(D6-A) -> Net-(D2-A)
- R47 pad 1: Net-(D7-A) -> Net-(D5-A)
- R48 pad 1: Net-(D8-A) -> Net-(D6-A)

Commit message: more routing
Parts:
- removed the D3 at (233.2, 118.5)
- removed the D5 at (235.5, 73.5)
- removed the D6 at (232.0, 73.5)
- removed D7, D8: LED_Small, LED_SMD:LED_0603_1608Metric_Pad1.05x0.95mm_HandSolder
- moved J10 101.8 mm to (270.5, 60.0), turned to 180 degrees
- moved J9 98.3 mm to (264.5, 65.0), turned to 180 degrees
- moved J11 94.7 mm to (247.5, 162.3), turned to 180 degrees
- moved J13 92.6 mm to (266.0, 48.3), turned to 180 degrees
- moved J12 90.6 mm to (233.0, 162.3), turned to 180 degrees
- moved D6 77.9 mm to (248.5, 73.0), turned to 90 degrees
- moved D5 68.0 mm to (239.0, 73.4), turned to 90 degrees
- moved D1 63.2 mm to (235.5, 73.4), turned to 90 degrees
- moved D2 60.5 mm to (232.0, 73.4), turned to 90 degrees
- moved D10 56.2 mm to (221.6, 136.5)
- moved D11 56.2 mm to (211.6, 137.6)
- moved D12 56.2 mm to (214.4, 141.5)
- moved D13 56.2 mm to (215.6, 135.0)
- moved D14 56.2 mm to (217.5, 124.0)
- moved D15 56.2 mm to (224.5, 124.0)
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Routing:
- net Electrode-: track 0.00 -> 49.5 mm
- net Safety+: track 0.00 -> 39.3 mm, vias 0 -> 2
- net Safety-: track 6.94 -> 42.7 mm, vias 0 -> 4
- net Current_Sense-: track 6.70 -> 39.8 mm, vias 0 -> 4
- net /Processor/TXD0: track 0.00 -> 24.9 mm, vias 0 -> 2
- net /Processor/RXDO: track 0.00 -> 24.7 mm, vias 0 -> 2
- net /Processor/SDA1: track 15.8 -> 38.3 mm
- net /Processor/SCL1: track 16.8 -> 34.3 mm
- net Electrode+: track 24.8 -> 41.7 mm
- net /Processor/SDA2: track 18.6 -> 34.8 mm
- net /HowlandPump/1IN-: track 0.21 -> 15.1 mm
- net /Processor/SCL2: track 19.2 -> 34.0 mm
- net Net-(D15-A): track 0.00 -> 7.63 mm
- net /HowlandPump/2IN+: track 14.0 -> 20.2 mm, vias 0 -> 2
- net Net-(U11-1IN_+): track 0.16 -> 6.21 mm
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Other:
- board size 30 x 100 mm -> 21.6 x 120.7 mm
